File: Kicad/Buck_TPS5430_Project/Buck_TPS5430_Project.kicad_sch (KiCad schematic)
At the start: 107 parts, among them J1 Vin, J2 GND, J3 Mode5V, J4 Mode12V, J5 Mode3.3-12V, J6 OUT+, J7 OUT-, J8 OUT3.3, J9 GND, Q1 APM4015P, U1 LMV358, U2 TPS5430DDA, U3 TPS5430DDA, U4 LM339, U5 LM7805R 5V 1.5A, U6 LD1117S33TR_SOT223, U7 TL431DBZ

Commit message: feat:PCB layout
Parts:
- removed C25, C26: 47u, symbol Device:C_Polarized_US
- removed C5, C6, C7, C8: 4.7u, symbol Device:C_Polarized_US
- removed D1: ZMM10 10V, symbol Device:D_Zener
- removed J1: Vin, symbol Connector_Generic:Conn_01x01
- removed J2, J9: GND, symbol Connector_Generic:Conn_01x01
- removed J6: OUT+, symbol Connector_Generic:Conn_01x01
- removed J7: OUT-, symbol Connector_Generic:Conn_01x01
- removed J8: OUT3.3, symbol Connector_Generic:Conn_01x01
- removed Q1: APM4015P, symbol Device:Q_PMOS
- removed R17: 5k 10%, symbol Device:R_Variable_US
- removed R19: 20m, symbol Device:R_Shunt_US
- removed R7: 100k, symbol Device:R_Variable_US
- removed U1: LMV358, symbol Amplifier_Operational:LMV358
- added C19: 47u, Capacitor_SMD:CP_Elec_6.3x7.7, symbol Device:C_Polarized_US
- added C5, C6, C7, C8: 4.7u, Capacitor_SMD:C_0805_2012Metric_Pad1.18x1.45mm_HandSolder, symbol Device:C
- added D1: ZMM10, Diode_SMD:D_MiniMELF, symbol Diode:ZMMxx
- added J1: Vin, TerminalBlock_Phoenix:TerminalBlock_Phoenix_MKDS-1,5-2-5.08_1x02_P5.08mm_Horizontal, symbol Connector:Screw_Terminal_01x02
- added J10: Vp, TerminalBlock_Phoenix:TerminalBlock_Phoenix_MKDS-1,5-2-5.08_1x02_P5.08mm_Horizontal, symbol Connector:Screw_Terminal_01x02
- added J6: 3.3V, TerminalBlock_Phoenix:TerminalBlock_Phoenix_MKDS-1,5-2-5.08_1x02_P5.08mm_Horizontal, symbol Connector:Screw_Terminal_01x02
- added J7: 5V, TerminalBlock_Phoenix:TerminalBlock_Phoenix_MKDS-1,5-2-5.08_1x02_P5.08mm_Horizontal, symbol Connector:Screw_Terminal_01x02
- added Q1: APM4015P, Package_TO_SOT_SMD:TO-252-2, symbol Transistor_FET:Q_PMOS_GDS
- added R13: 1.2k 1%, Resistor_SMD:R_0805_2012Metric_Pad1.20x1.40mm_HandSolder, symbol Device:R_US
- added R19: 20m 1%, Resistor_SMD:R_2512_6332Metric_Pad1.40x3.35mm_HandSolder, symbol Device:R_US
- added R9: 3k 1%, Resistor_SMD:R_0805_2012Metric_Pad1.20x1.40mm_HandSolder, symbol Device:R_US
- added RV1: 100k 10%, Potentiometer_THT:Potentiometer_Bourns_3296W_Vertical, symbol Device:R_Potentiometer_Trim_US
- added RV2: 5k 10%, Potentiometer_THT:Potentiometer_Bourns_3296W_Vertical, symbol Device:R_Potentiometer_Trim_US
- added TP22: TP_7.3V, TestPoint:TestPoint_Pad_D1.0mm, symbol Connector:TestPoint
- added TP23, TP24: TP_GND, TestPoint:TestPoint_Pad_D1.0mm, symbol Connector:TestPoint
- added U1: LM358, Package_SO:SOIC-8_3.9x4.9mm_P1.27mm, symbol Amplifier_Operational:LM358
- C1, C2, C20, C21, C22, C23, C3, C4: footprint (none) -> Capacitor_SMD:CP_Elec_6.3x7.7; Link (none) -> https://www.thegioiic.com/tu-nhom-smd-47uf-50v-6-3x7-7mm
- C10, C13, C16: footprint (none) -> Capacitor_SMD:C_0805_2012Metric_Pad1.18x1.45mm_HandSolder; Link (none) -> https://www.thegioiic.com/tu-gom-0805-10nf-50v
- C11, C12: footprint (none) -> Capacitor_SMD:C_0805_2012Metric_Pad1.18x1.45mm_HandSolder; Link (none) -> https://www.thegioiic.com/tu-gom-1206-100pf-50v
- C14, C15, C17, C18: footprint (none) -> Capacitor_SMD:C_0805_2012Metric_Pad1.18x1.45mm_HandSolder; Link (none) -> https://www.thegioiic.com/tu-gom-0805-100nf-0-1uf-50v
- C24: renamed from C19; footprint (none) -> Capacitor_SMD:C_0805_2012Metric_Pad1.18x1.45mm_HandSolder; Link (none) -> https://www.thegioiic.com/tu-gom-0805-100nf-0-1uf-50v
- C25: renamed from C24; footprint (none) -> Capacitor_SMD:C_0805_2012Metric_Pad1.18x1.45mm_HandSolder; Link (none) -> https://www.thegioiic.com/tu-gom-0805-100nf-0-1uf-50v
- C26: renamed from C28; footprint (none) -> Capacitor_SMD:C_0805_2012Metric_Pad1.18x1.45mm_HandSolder; Link (none) -> https://www.thegioiic.com/tu-gom-0805-100nf-0-1uf-50v
- C27: renamed from C30; footprint (none) -> Capacitor_SMD:C_0805_2012Metric_Pad1.18x1.45mm_HandSolder; Link (none) -> https://www.thegioiic.com/tu-gom-0805-10uf-25v
- C28: renamed from C27; footprint (none) -> Capacitor_SMD:C_0805_2012Metric_Pad1.18x1.45mm_HandSolder; Link (none) -> https://www.thegioiic.com/tu-gom-0805-330nf-50v
- C29: renamed from C31; footprint (none) -> Capacitor_SMD:C_0805_2012Metric_Pad1.18x1.45mm_HandSolder; Link (none) -> https://www.thegioiic.com/tu-gom-0805-100nf-0-1uf-50v
- C30: renamed from C29; footprint (none) -> Capacitor_SMD:C_0805_2012Metric_Pad1.18x1.45mm_HandSolder; Link (none) -> https://www.thegioiic.com/tu-gom-0805-100nf-0-1uf-50v
- C9: footprint (none) -> Capacitor_SMD:C_0805_2012Metric_Pad1.18x1.45mm_HandSolder; Link (none) -> https://www.thegioiic.com/tu-gom-0805-1uf-25v
- D2, D3, D4: footprint (none) -> Diode_SMD:D_SMC; Link (none) -> https://dientutuonglai.com/b340a-diode-schottky-40v-3a-sma-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
- D5, D6, D7, D8, D9: footprint (none) -> LED_SMD:LED_0805_2012Metric_Pad1.15x1.40mm_HandSolder; Link (none) -> https://www.thegioiic.com/led-do-0805-dan-smd-trong-suot-ha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
- F1: footprint (none) -> Capacitor_THT:C_Disc_D11.0mm_W5.0mm_P5.00mm; Link (none) -> https://www.thegioiic.com/uf300-cau-chi-tu-phuc-hoi-30v-3a
- J3, J4, J5: footprint (none) -> Connector_PinHeader_2.54mm:PinHeader_1x02_P2.54mm_Vertical; Link (none) -> https://www.thegioiic.com/jumper-2-54mm-ngan-mach-6-5mm-mau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
- L1: value 20-25u -> 22u; footprint (none) -> Inductor_SMD:L_Coilcraft_MSS1038-XXX; Link (none) -> https://www.thegioiic.com/cuon-cam-dan-smd-cdrh104-1038-220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
- L2: value 30-50u -> 33u; footprint (none) -> Inductor_SMD:L_Coilcraft_MSS1278-XXX; Link (none) -> https://www.thegioiic.com/cuon-cam-dan-smd-cdrh127-1280-330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
- R1: footprint (none) -> Resistor_SMD:R_0805_2012Metric_Pad1.20x1.40mm_HandSolder; Link (none) -> https://www.thegioiic.com/dien-tro-4-7-kohm-0805-1-
- R10, R11, R12: value ~ -> 330 5%; footprint (none) -> Resistor_SMD:R_0805_2012Metric_Pad1.20x1.40mm_HandSolder; Link (none) -> https://www.thegioiic.com/dien-tro-330-ohm-0805-5-
- R14: renamed from R13; value 1.13k -> 20k 1%; footprint (none) -> Resistor_SMD:R_0805_2012Metric_Pad1.20x1.40mm_HandSolder; Link (none) -> https://www.thegioiic.com/dien-tro-20-kohm-0805-1-
- R15: renamed from R14; value 10k -> 10k 1%; footprint (none) -> Resistor_SMD:R_0805_2012Metric_Pad1.20x1.40mm_HandSolder; Link (none) -> https://www.thegioiic.com/dien-tro-10-kohm-0805-1-
- R16: renamed from R15; footprint (none) -> Resistor_SMD:R_0805_2012Metric_Pad1.20x1.40mm_HandSolder; Link (none) -> https://www.thegioiic.com/dien-tro-2-kohm-0805-1-
- R17: renamed from R16; footprint (none) -> Resistor_SMD:R_0805_2012Metric_Pad1.20x1.40mm_HandSolder; Link (none) -> https://www.thegioiic.com/dien-tro-10-kohm-0805-1-
- R18, R2, R3: footprint (none) -> Resistor_SMD:R_0805_2012Metric_Pad1.20x1.40mm_HandSolder; Link (none) -> https://www.thegioiic.com/dien-tro-1-kohm-0805-1-
- R20: value ~ -> 220; footprint (none) -> Resistor_SMD:R_0805_2012Metric_Pad1.20x1.40mm_HandSolder; Link (none) -> https://www.thegioiic.com/dien-tro-220-ohm-0805-1-
- R21: footprint (none) -> Resistor_SMD:R_0805_2012Metric_Pad1.20x1.40mm_HandSolder; Link (none) -> https://www.thegioiic.com/dien-tro-12-kohm-0805-1-
- R22: footprint (none) -> Resistor_SMD:R_0805_2012Metric_Pad1.20x1.40mm_HandSolder; Link (none) -> https://www.thegioiic.com/dien-tro-1-2-kohm-0805-1-
- R23: renamed from R24; value ~ -> 330 5%; footprint (none) -> Resistor_SMD:R_0805_2012Metric_Pad1.20x1.40mm_HandSolder; Link (none) -> https://www.thegioiic.com/dien-tro-330-ohm-0805-5-
- R24: renamed from R23; footprint (none) -> Resistor_SMD:R_0805_2012Metric_Pad1.20x1.40mm_HandSolder; Link (none) -> https://www.thegioiic.com/dien-tro-10-kohm-0805-1-
- R25: renamed from R26; value ~ -> 330 5%; footprint (none) -> Resistor_SMD:R_0805_2012Metric_Pad1.20x1.40mm_HandSolder; Link (none) -> https://www.thegioiic.com/dien-tro-330-ohm-0805-5-
- R26: renamed from R25; footprint (none) -> Resistor_SMD:R_0805_2012Metric_Pad1.20x1.40mm_HandSolder; Link (none) -> https://www.thegioiic.com/dien-tro-1-5-kohm-0805-1-
- R4, R5: footprint (none) -> Resistor_SMD:R_0805_2012Metric_Pad1.20x1.40mm_HandSolder; Link (none) -> https://www.thegioiic.com/dien-tro-49-9-kohm-0805-1-
- R6: footprint (none) -> Resistor_SMD:R_0805_2012Metric_Pad1.20x1.40mm_HandSolder; Link (none) -> https://www.thegioiic.com/dien-tro-10-kohm-0805-1-
- R7: renamed from R8; footprint (none) -> Resistor_SMD:R_0805_2012Metric_Pad1.20x1.40mm_HandSolder; Link (none) -> https://www.thegioiic.com/dien-tro-100-ohm-0805-1-
- R8: renamed from R9; value 3.23k -> 220 1%; footprint (none) -> Resistor_SMD:R_0805_2012Metric_Pad1.20x1.40mm_HandSolder; Link (none) -> https://www.thegioiic.com/dien-tro-220-ohm-0805-1-
- TP1, TP10, TP11, TP12, TP13, TP14, TP15, TP2, TP20, TP21, TP3, TP4, TP5, TP6, TP7, TP8, TP9: footprint (none) -> TestPoint:TestPoint_Pad_D1.0mm
- TP16: renamed from TP18; footprint (none) -> TestPoint:TestPoint_Pad_D1.0mm
- TP17: renamed from TP16; footprint (none) -> TestPoint:TestPoint_Pad_D1.0mm
- TP18: renamed from TP19; footprint (none) -> TestPoint:TestPoint_Pad_D1.0mm
- TP19: renamed from TP17; footprint (none) -> TestPoint:TestPoint_Pad_D1.0mm
- U2, U3: Link (none) -> https://www.thegioiic.com/tps5430ddar-ic-dieu-chinh-giam-ap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
- U4: footprint (none) -> Package_SO:SOIC-14_3.9x8.7mm_P1.27mm; Link (none) -> https://www.thegioiic.com/lm339dr-ic-quad-comparator-cmos-t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
- U5: renamed from U6; Link (none) -> https://www.thegioiic.com/ld1117s33ctr-ic-on-ap-3-3v-800ma-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
- U6: renamed from U5; footprint Package_TO_SOT_SMD:SOT-223-3_TabPin2 -> Package_TO_SOT_SMD:TO-263-3_TabPin2; Link (none) -> https://www.thegioiic.com/lm7805r-ic-on-ap-5v-1-5a-to-263
- U7: Link (none) -> https://www.thegioiic.com/tl431-ic-tham-chieu-dien-ap-2-5-3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
Connections:
- net ENA is gone; now on net ENA2: C16.1, D2.1 (K), U4.13
- net Shunt+ is gone; now on net OUT-: R2.1
- net Shunt- is gone; now on net GND: R3.1
- net +5V: now also U6.3 (VO), J7.1 (Pin_1), U1.8 (V+); no longer U6.2 (VO)
- net 7.326V: now also U6.1 (VI), TP22.1; no longer U6.3 (VI)
- net GND: now also U6.2 (GND), C19.2, C5.2, C6.2, C7.2, C8.2, J1.1 (Pin_2), J6.2 (Pin_2), J7.2 (Pin_2), R13.2, R19.2, R9.2, RV1.3, TP23.1, TP24.1, U1.4 (V-); no longer R8.2, U6.1 (GND)
- net OUT+: now also C19.1, J10.1 (Pin_1)
- net OUT-: now also J10.2 (Pin_2), R19.1
- net VIN: now also C5.1, C6.1, C7.1, C8.1, D1.1 (K), Q1.3 (S)
- net VSENSE: now also U1.5 (+); no longer R15.2, R16.2, TP10.1, U2.4 (VSENSE)
- net at C29.2, U4.4 (-), U4.6 (-): now also U1.6 (-), U1.7
- net at R3.2, R5.1: now also U1.2 (-)
- net at F1.2: now also Q1.2 (D)
- net at R1.1: now also D1.2 (A), Q1.1 (G)
- net at C10.1, C9.2, R6.1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: now also RV1.1, RV1.2
- net at C13.1, R5.2, TP7.1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: now also U1.1
- net at R18.2: now also RV2.3
- net at R2.2, R4.1: now also U1.3 (+)
- net at C27.2, TP16.1, U5.2 (VO): now also J6.1 (Pin_1)
- net at F1.1: now also J1.2 (Pin_1)
- net at J4.2 (Pin_2), R14.1: now also R13.1
- net at J5.2 (Pin_2): now also RV2.1, RV2.2
- new net: R15.2, R16.2, TP10.1, U2.4 (VSENSE)
- new net: R8.2, R9.1
Other:
- moved on the sheet: C11, C24, C25, C28, C30, D5, J3, J4, R10, R14, R18, R21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
