File: Kicad/Buck_TPS5430/Buck_TPS5430.kicad_sch (KiCad schematic)
At the start: 109 parts, among them J1 Vin, J10 Vp, J3 Mode5V, J4 Mode12V, J5 Mode3.3-12V, J6 3.3V, J7 5V, Q1 APM4015P, U1 LM358, U2 TPS5430DDA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

Commit message: feat: COMPLETE PCB Layout
Parts:
- added H1, H2, H3, H4: MountingHole, MountingHole:MountingHole_3.2mm_M3, symbol Mechanical:MountingHole
- J1, J10, J6, J7: Link (none) -> https://www.thegioiic.com/kf301-2-v-domino-2-chan-thang-5-0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
Connections:
- net OUT+: now also J10.2 (Pin_1); no longer J10.1 (Pin_1)
- net OUT-: now also J10.1 (Pin_2); no longer J10.2 (Pin_2)
- net PH2: now reaches C15.2, D4.1 (K), L2.1, TP13.1, U3.8 (PH)
- net PH1: now reaches C14.2, D3.1 (K), L1.1, TP12.1, U2.8 (PH)
